File: kicad/F1_anemometers.sch (KiCad schematic (older format))
At the start: 22 parts, among them U1 MCP6244

Commit message: nothing
Parts:
- R10, R2, R3, R4, R5, R6, R7, R9: Tolerance (none) -> 1%; Tolérance 1% -> (none)
Changed lines of the file:
@@
 F 3 "~" H 3750 4850 30  0000 C CNN
 F 4 "0.125W" V 3750 4850 60  0001 C CNN "Puissance"
-F 5 "1%" V 3750 4850 60  0001 C CNN "Tolérance"
+F 5 "1%" V 3750 4850 60  0001 C CNN "Tolerance"
 	1    3750 4850
 	-1   0    0    1
@@
 F 3 "~" H 5950 6425 30  0000 C CNN
 F 4 "0.125W" V 5950 6425 60  0001 C CNN "Puissance"
-F 5 "1%" V 5950 6425 60  0001 C CNN "Tolérance"
+F 5 "1%" V 5950 6425 60  0001 C CNN "Tolerance"
 	1    5950 6425
 	1    0    0    -1
@@
 F 3 "~" H 6450 6075 30  0000 C CNN
 F 4 "0.125W" V 6450 6075 60  0001 C CNN "Puissance"
-F 5 "1%" V 6450 6075 60  0001 C CNN "Tolérance"
+F 5 "1%" V 6450 6075 60  0001 C CNN "Tolerance"
 	1    6450 6075
 	0    -1   -1   0
@@
 F 3 "~" H 6275 3175 30  0000 C CNN
 F 4 "0.125W" V 6275 3175 60  0001 C CNN "Puissance"
-F 5 "1%" V 6275 3175 60  0001 C CNN "Tolérance"
+F 5 "1%" V 6275 3175 60  0001 C CNN "Tolerance"
 	1    6275 3175
 	0    -1   -1   0
@@
 F 3 "~" H 5750 3525 30  0000 C CNN
 F 4 "0.125W" V 5750 3525 60  0001 C CNN "Puissance"
-F 5 "1%" V 5750 3525 60  0001 C CNN "Tolérance"
+F 5 "1%" V 5750 3525 60  0001 C CNN "Tolerance"
 	1    5750 3525
 	1    0    0    -1
@@
 F 3 "~" H 3700 1900 30  0000 C CNN
 F 4 "0.125W" V 3700 1900 60  0001 C CNN "Puissance"
-F 5 "1%" V 3700 1900 60  0001 C CNN "Tolérance"
+F 5 "1%" V 3700 1900 60  0001 C CNN "Tolerance"
 	1    3700 1900
 	-1   0    0    1
@@
 F 3 "~" H 4350 3250 30  0000 C CNN
 F 4 "0.125W" V 4350 3250 60  0001 C CNN "Puissance"
-F 5 "1%" V 4350 3250 60  0001 C CNN "Tolérance"
+F 5 "1%" V 4350 3250 60  0001 C CNN "Tolerance"
 	1    4350 3250
 	1    0    0    -1
@@
 F 3 "~" H 4400 6300 30  0000 C CNN
 F 4 "0.125W" V 4400 6300 60  0001 C CNN "Puissance"
-F 5 "1%" V 4400 6300 60  0001 C CNN "Tolérance"
+F 5 "1%" V 4400 6300 60  0001 C CNN "Tolerance"
 	1    4400 6300
 	1    0    0    -1
