File: kicad/F2_windvane.sch (KiCad schematic (older format))
At the start: 7 parts, among them U1 MCP6244

Commit message: nothing
Parts:
- R11, R12: Tolerance (none) -> 1%; Tolérance 1% -> (none)
Changed lines of the file:
@@
 F 3 "~" H 4050 2550 30  0000 C CNN
 F 4 "0.125W" V 4050 2550 60  0001 C CNN "Puissance"
-F 5 "1%" V 4050 2550 60  0001 C CNN "Tolérance"
+F 5 "1%" V 4050 2550 60  0001 C CNN "Tolerance"
 	1    4050 2550
 	1    0    0    -1
@@
 F 3 "~" H 5150 3300 30  0000 C CNN
 F 4 "0.125W" V 5150 3300 60  0001 C CNN "Puissance"
-F 5 "1%" V 5150 3300 60  0001 C CNN "Tolérance"
+F 5 "1%" V 5150 3300 60  0001 C CNN "Tolerance"
 	1    5150 3300
 	0    -1   -1   0
