File: kicad/F3_Voltage_sensors.sch (KiCad schematic (older format))
At the start: 19 parts, among them U1 MCP6244, U2 MCP6242

Commit message: nothing
Parts:
- R17, R18, R19, R20, R21, R22: Tolerance (none) -> 1%; Tolérance 1% -> (none)
Changed lines of the file:
@@
 F 3 "~" H 7350 4550 30  0000 C CNN
 F 4 "0.125W" V 7350 4550 60  0001 C CNN "Puissance"
-F 5 "1%" V 7350 4550 60  0001 C CNN "Tolérance"
+F 5 "1%" V 7350 4550 60  0001 C CNN "Tolerance"
 	1    7350 4550
 	1    0    0    -1
@@
 F 3 "~" H 7500 3400 30  0000 C CNN
 F 4 "0.125W" V 7500 3400 60  0001 C CNN "Puissance"
-F 5 "1%" V 7500 3400 60  0001 C CNN "Tolérance"
+F 5 "1%" V 7500 3400 60  0001 C CNN "Tolerance"
 	1    7500 3400
 	1    0    0    -1
@@
 F 3 "~" H 1825 4325 30  0000 C CNN
 F 4 "0.125W" V 1825 4325 60  0001 C CNN "Puissance"
-F 5 "1%" V 1825 4325 60  0001 C CNN "Tolérance"
+F 5 "1%" V 1825 4325 60  0001 C CNN "Tolerance"
 	1    1825 4325
 	1    0    0    -1
@@
 F 3 "~" H 1825 3375 30  0000 C CNN
 F 4 "0.125W" V 1825 3375 60  0001 C CNN "Puissance"
-F 5 "1%" V 1825 3375 60  0001 C CNN "Tolérance"
+F 5 "1%" V 1825 3375 60  0001 C CNN "Tolerance"
 	1    1825 3375
 	1    0    0    -1
@@
 F 3 "~" H 7500 3950 30  0000 C CNN
 F 4 "0.125W" V 7500 3950 60  0001 C CNN "Puissance"
-F 5 "1%" V 7500 3950 60  0001 C CNN "Tolérance"
+F 5 "1%" V 7500 3950 60  0001 C CNN "Tolerance"
 	1    7500 3950
 	1    0    0    -1
@@
 F 3 "~" H 7600 4550 30  0000 C CNN
 F 4 "0.125W" V 7600 4550 60  0001 C CNN "Puissance"
-F 5 "1%" V 7600 4550 60  0001 C CNN "Tolérance"
+F 5 "1%" V 7600 4550 60  0001 C CNN "Tolerance"
 	1    7600 4550
 	1    0    0    -1
