File: kicad/F4_Current_sensors.sch (KiCad schematic (older format))
At the start: 26 parts, among them U3 MCP6244

Commit message: nothing
Parts:
- R23, R24, R25, R26, R27, R28, R29, R30, R31, R32, R33, R34: Tolerance (none) -> 1%; Tolérance 1% -> (none)
Changed lines of the file:
@@
 F 3 "~" H 2375 2325 30  0000 C CNN
 F 4 "0.125W" V 2375 2325 60  0001 C CNN "Puissance"
-F 5 "1%" V 2375 2325 60  0001 C CNN "Tolérance"
+F 5 "1%" V 2375 2325 60  0001 C CNN "Tolerance"
 	1    2375 2325
 	1    0    0    -1
@@
 F 3 "~" H 3025 2300 30  0000 C CNN
 F 4 "0.125W" V 3025 2300 60  0001 C CNN "Puissance"
-F 5 "1%" V 3025 2300 60  0001 C CNN "Tolérance"
+F 5 "1%" V 3025 2300 60  0001 C CNN "Tolerance"
 	1    3025 2300
 	1    0    0    -1
@@
 F 3 "~" H 3025 2900 30  0000 C CNN
 F 4 "0.125W" V 3025 2900 60  0001 C CNN "Puissance"
-F 5 "1%" V 3025 2900 60  0001 C CNN "Tolérance"
+F 5 "1%" V 3025 2900 60  0001 C CNN "Tolerance"
 	1    3025 2900
 	1    0    0    -1
@@
 F 3 "~" H 2350 5200 30  0000 C CNN
 F 4 "0.125W" V 2350 5200 60  0001 C CNN "Puissance"
-F 5 "1%" V 2350 5200 60  0001 C CNN "Tolérance"
+F 5 "1%" V 2350 5200 60  0001 C CNN "Tolerance"
 	1    2350 5200
 	1    0    0    -1
@@
 F 3 "~" H 3000 5175 30  0000 C CNN
 F 4 "0.125W" V 3000 5175 60  0001 C CNN "Puissance"
-F 5 "1%" V 3000 5175 60  0001 C CNN "Tolérance"
+F 5 "1%" V 3000 5175 60  0001 C CNN "Tolerance"
 	1    3000 5175
 	1    0    0    -1
@@
 F 3 "~" H 3000 5775 30  0000 C CNN
 F 4 "0.125W" V 3000 5775 60  0001 C CNN "Puissance"
-F 5 "1%" V 3000 5775 60  0001 C CNN "Tolérance"
+F 5 "1%" V 3000 5775 60  0001 C CNN "Tolerance"
 	1    3000 5775
 	1    0    0    -1
@@
 F 3 "~" H 7450 2325 30  0000 C CNN
 F 4 "0.125W" V 7450 2325 60  0001 C CNN "Puissance"
-F 5 "1%" V 7450 2325 60  0001 C CNN "Tolérance"
+F 5 "1%" V 7450 2325 60  0001 C CNN "Tolerance"
 	1    7450 2325
 	1    0    0    -1
@@
 F 3 "~" H 8100 2300 30  0000 C CNN
 F 4 "0.125W" V 8100 2300 60  0001 C CNN "Puissance"
-F 5 "1%" V 8100 2300 60  0001 C CNN "Tolérance"
+F 5 "1%" V 8100 2300 60  0001 C CNN "Tolerance"
 	1    8100 2300
 	1    0    0    -1
@@
 F 3 "~" H 8100 2900 30  0000 C CNN
 F 4 "0.125W" V 8100 2900 60  0001 C CNN "Puissance"
-F 5 "1%" V 8100 2900 60  0001 C CNN "Tolérance"
+F 5 "1%" V 8100 2900 60  0001 C CNN "Tolerance"
 	1    8100 2900
 	1    0    0    -1
@@
 F 3 "~" H 7375 5175 30  0000 C CNN
 F 4 "0.125W" V 7375 5175 60  0001 C CNN "Puissance"
-F 5 "1%" V 7375 5175 60  0001 C CNN "Tolérance"
+F 5 "1%" V 7375 5175 60  0001 C CNN "Tolerance"
 	1    7375 5175
 	1    0    0    -1
@@
 F 3 "~" H 8025 5150 30  0000 C CNN
 F 4 "0.125W" V 8025 5150 60  0001 C CNN "Puissance"
-F 5 "1%" V 8025 5150 60  0001 C CNN "Tolérance"
+F 5 "1%" V 8025 5150 60  0001 C CNN "Tolerance"
 	1    8025 5150
 	1    0    0    -1
@@
 F 3 "~" H 8025 5750 30  0000 C CNN
 F 4 "0.125W" V 8025 5750 60  0001 C CNN "Puissance"
-F 5 "1%" V 8025 5750 60  0001 C CNN "Tolérance"
+F 5 "1%" V 8025 5750 60  0001 C CNN "Tolerance"
 	1    8025 5750
 	1    0    0    -1
