File: kicad/F5_temperature.sch (KiCad schematic (older format))
At the start: 10 parts, among them U502 LMV358, U601 LMV358

Commit message: nothing
Parts:
- NTC601: Tolerance (none) -> 5%; Tolérance 5% -> (none)
- R601, R603, R604, R605, R606: Tolerance (none) -> 1%; Tolérance 1% -> (none)
Changed lines of the file:
@@
 F 2 "Discret:R4" H 4100 4050 60  0001 C CNN
 F 3 "~" H 4100 4050 60  0000 C CNN
-F 4 "5%" V 4100 4050 60  0001 C CNN "Tolérance"
+F 4 "5%" V 4100 4050 60  0001 C CNN "Tolerance"
 	1    4100 4050
 	1    0    0    -1
@@
 F 3 "~" H 4100 3000 30  0000 C CNN
 F 4 "0.125W" V 4100 3000 60  0001 C CNN "Puissance"
-F 5 "1%" V 4100 3000 60  0001 C CNN "Tolérance"
+F 5 "1%" V 4100 3000 60  0001 C CNN "Tolerance"
 	1    4100 3000
 	1    0    0    -1
@@
 F 2 "Discret:R4" V 5130 4250 30  0001 C CNN
 F 3 "~" H 5200 4250 30  0000 C CNN
-F 4 "1%" V 5200 4250 60  0001 C CNN "Tolérance"
+F 4 "1%" V 5200 4250 60  0001 C CNN "Tolerance"
 F 5 "1/8W" V 5200 4250 60  0001 C CNN "Puissance"
 	1    5200 4250
@@
 F 2 "Discret:R4" V 5830 4700 30  0001 C CNN
 F 3 "~" H 5900 4700 30  0000 C CNN
-F 4 "1%" V 5900 4700 60  0001 C CNN "Tolérance"
+F 4 "1%" V 5900 4700 60  0001 C CNN "Tolerance"
 F 5 "1/8W" V 5900 4700 60  0001 C CNN "Puissance"
 	1    5900 4700
@@
 F 2 "Discret:R4" V 7230 3700 30  0001 C CNN
 F 3 "~" H 7300 3700 30  0000 C CNN
-F 4 "1%" V 7300 3700 60  0001 C CNN "Tolérance"
+F 4 "1%" V 7300 3700 60  0001 C CNN "Tolerance"
 F 5 "1/8W" V 7300 3700 60  0001 C CNN "Puissance"
 	1    7300 3700
@@
 F 2 "Discret:R4" V 8430 4700 30  0001 C CNN
 F 3 "~" H 8500 4700 30  0000 C CNN
-F 4 "1%" V 8500 4700 60  0001 C CNN "Tolérance"
+F 4 "1%" V 8500 4700 60  0001 C CNN "Tolerance"
 F 5 "1/8W" V 8500 4700 60  0001 C CNN "Puissance"
 	1    8500 4700
