File: kicad/shield.sch (KiCad schematic (older format))
At the start: 26 parts

Commit message: nothing
Parts:
- R1: Tolerance (none) -> 1%; Tolérance 1% -> (none)
Changed lines of the file:
@@
 F 3 "~" H 3250 7150 30  0000 C CNN
 F 4 "0.125W" V 3250 7150 60  0001 C CNN "Puissance"
-F 5 "1%" V 3250 7150 60  0001 C CNN "Tolérance"
+F 5 "1%" V 3250 7150 60  0001 C CNN "Tolerance"
 	1    3250 7150
 	0    1    1    0
